File: hp35battery.kicad_sch (KiCad schematic)
At the start: 29 parts, among them J1 USB_B_Micro, J2 PAD+, J3 PAD-, Q1 2N7002, U1 TP4056, U2 MIC5205YM5, U3 MAX40200AUK, U4 DW01A, U5 FS8205

Commit message: Further calc and schematic update
Parts:
- R1: value 5k -> 4k
- R4: value 220k -> 300k
- R5: value 100k -> 160k
- U2: value MIC5205YM5 -> TPS73101
- U4: value DW01A -> S-8261ABJMD
Other:
- note added: "--> 80~125mA (UNPLUGGED, ON) <-- 50mA (<16V) (PLUGGED IN)"
- note added: "2.92~3.55V"
- note added: "2.97~3.60V"
- note added: "3.00~4.26V"
- note added: "30mOhm (negligible drop)"
- note added: "<30mV drop"
- note added: "BATTERY R1 ICHG TCHG R8 ICHG TCHG TRUN (USB) (USB) (HP) (HP) 2000 mAh 3k0 400mA 5H 22k 48mA 42H 1500 mAh 3k9 308mA 5H 22k 46.3mA 33H 16h (see spreadsheet) 1000 mAh 5k6 214mA 5H 20k 46.9mA 22H"
- note added: "Low battery lamp at 3.50V"
- note added: "REV1 ADD Q1,R8,R9 REV1.1 U2=TPS73101, U4=S-8261ABJMD, R4=300k, R5=160k"
- note removed: "--> 85~110mA (UNPLUGGED, ON) <-- 50mA (<16V) (PLUGGED IN)"
- note removed: "2.29~3.95V"
- note removed: "2.34~4.00V"
- note removed: "2.50~4.30V"
- note removed: "<160mV drop"
- note removed: "BATTERY R1 ICHG TCHG R8 ICHG TCHG TRUN (USB) (USB) (HP) (HP) (85%) 2000 mAh 3k0 400mA 5H 22k 48mA 42H 17H 1500 mAh 4k0 300mA 5H 22k 46mA 33H 12H 1000 mAh 6k0 200mA 5H 20k 46mA 22H 8H"
- note removed: "Low battery lamp at 3.50V REG NOREG VOUT 3.50 3.50 VREG 3.55 3.55 B+ 3.71 3.55 Usable 85% 95%"
Changed lines of the file:
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@@
     (stroke (width 0) (type default))
   )
-  (text "2.50~4.30V" (at 165.1 88.9 0)
-    (effects (font (size 1.27 1.27)) (justify left bottom))
-  )
-  (text "BATTERY		R1		ICHG	TCHG	R8		ICHG	TCHG	TRUN\n					(USB)	(USB)			(HP)	(HP)	(85%)\n2000 mAh	3k0		400mA	5H		22k		48mA	42H		17H\n1500 mAh	4k0		300mA	5H		22k		46mA	33H		12H\n1000 mAh	6k0		200mA	5H		20k		46mA	22H		8H"
+  (text "3.00~4.26V" (at 165.1 88.9 0)
+    (effects (font (size 1.27 1.27)) (justify left bottom))
+  )
+  (text "BATTERY		R1		ICHG	TCHG	R8		ICHG	TCHG	TRUN\n					(USB)	(USB)			(HP)	(HP)	\n2000 mAh	3k0		400mA	5H		22k		48mA	42H		\n1500 mAh	3k9		308mA	5H		22k		46.3mA	33H		16h (see spreadsheet)\n1000 mAh	5k6		214mA	5H		20k		46.9mA	22H		"
     (at 86.36 52.07 0)
     (effects (font (size 1.27 1.27)) (justify left bottom))
   )
-  (text "--> 85~110mA (UNPLUGGED, ON)\n<-- 50mA (<16V) (PLUGGED IN)"
+  (text "--> 80~125mA (UNPLUGGED, ON)\n<-- 50mA (<16V) (PLUGGED IN)"
     (at 250.19 87.63 0)
     (effects (font (size 1.27 1.27)) (justify left bottom))
@@
     (effects (font (size 1.27 1.27)) (justify left bottom))
   )
-  (text "2.34~4.00V" (at 203.2 76.2 0)
+  (text "2.97~3.60V" (at 203.2 76.2 0)
     (effects (font (size 1.27 1.27)) (justify left bottom))
   )
@@
     (effects (font (size 1.27 1.27)) (justify left bottom))
   )
-  (text "<160mV drop" (at 176.53 71.12 0)
+  (text "<30mV drop" (at 176.53 71.12 0)
     (effects (font (size 1.27 1.27)) (justify left bottom))
   )
@@
     (effects (font (size 1.27 1.27)) (justify left bottom))
   )
-  (text "2.29~3.95V" (at 254 77.47 0)
+  (text "2.92~3.55V" (at 254 77.47 0)
     (effects (font (size 1.27 1.27)) (justify left bottom))
   )
@@
     (effects (font (size 1.27 1.27)) (justify left bottom))
   )
+  (text "30mOhm (negligible drop)" (at 50.8 176.53 0)
+    (effects (font (size 1.27 1.27)) (justify left bottom))
+  )
   (text "0.04mA (HP)" (at 93.98 78.74 0)
     (effects (font (size 1.27 1.27)) (justify left bottom))
@@
     (effects (font (size 1.27 1.27)) (justify left bottom))
   )
-  (text "Low battery lamp at 3.50V\n\n		REG			NOREG\n\nVOUT	3.50		3.50\nVREG	3.55		3.55\nB+		3.71		3.55\nUsable	85%        	95%"
-    (at 234.95 39.37 0)
+  (text "REV1 ADD Q1,R8,R9\n\nREV1.1 U2=TPS73101, U4=S-8261ABJMD, R4=300k, R5=160k"
+    (at 113.03 194.31 0)
+    (effects (font (size 1.27 1.27)) (justify left bottom))
+  )
+  (text "Low battery lamp at 3.50V" (at 252.73 92.71 0)
     (effects (font (size 1.27 1.27)) (justify left bottom))
   )
@@
       (effects (font (size 1.27 1.27)) (justify left))
     )
-    (property "Value" "220k" (at 203.2 88.9 0)
+    (property "Value" "300k" (at 203.2 88.9 0)
       (effects (font (size 1.27 1.27)) (justify left))
     )
@@
   (symbol (lib_id "Regulator_Linear:MIC5205YM5") (at 181.61 83.82 0) (unit 1)
     (in_bom yes) (on_board yes) (dnp no) (fields_autoplaced)
-    (property "Reference" "U2" (at 181.61 73.66 0)
-      (effects (font (size 1.27 1.27)))
-    )
-    (property "Value" "MIC5205YM5" (at 181.61 76.2 0)
+    (property "Reference" "U2" (at 181.61 74.93 0)
+      (effects (font (size 1.27 1.27)))
+    )
+    (property "Value" "TPS73101" (at 181.61 77.47 0)
       (effects (font (size 1.27 1.27)))
     )
@@
       (effects (font (size 1.27 1.27)) (justify right))
     )
-    (property "Value" "5k" (at 110.49 82.55 0)
+    (property "Value" "4k" (at 110.49 82.55 0)
       (effects (font (size 1.27 1.27)) (justify right))
     )
@@
       (effects (font (size 1.27 1.27)) (justify left))
     )
-    (property "Value" "100k" (at 203.2 99.06 0)
+    (property "Value" "160k" (at 203.2 99.06 0)
       (effects (font (size 1.27 1.27)) (justify left))
     )
@@
       (effects (font (size 1.27 1.27)))
     )
-    (property "Value" "DW01A" (at 60.96 123.19 0)
-      (effects (font (size 1.27 1.27)))
-    )
+    (property "Value" "S-8261ABJMD" (at 60.96 123.19 0)
+      (effects (font (size 1.27 1.27)))
+    )

Commit message: Schematic plot
Other:
- note added: "REV1 ADD Q1,R8,R9 REV1.1 U2=TPS73101, U4=S-8261ABJMD, R4=300k, R5=160k, update notes"
- note removed: "REV1 ADD Q1,R8,R9 REV1.1 U2=TPS73101, U4=S-8261ABJMD, R4=300k, R5=160k"
Changed lines of the file:
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@@
   (title_block
     (title "HP BATTERY")
-    (date "2023-08-15")
-    (rev "1")
+    (date "2023-08-21")
+    (rev "1.1")
     (company "GR")
+    (comment 1 "https://github.com/grob6000/hpbattery")
   )
   (junction (at 116.84 104.14) (diameter 0) (color 0 0 0 0)
@@
     (effects (font (size 1.27 1.27)) (justify left bottom))
   )
-  (text "REV1 ADD Q1,R8,R9\n\nREV1.1 U2=TPS73101, U4=S-8261ABJMD, R4=300k, R5=160k"
-    (at 113.03 194.31 0)
-    (effects (font (size 1.27 1.27)) (justify left bottom))
-  )
+  (text "REV1 ADD Q1,R8,R9\n\nREV1.1 U2=TPS73101, U4=S-8261ABJMD, R4=300k, R5=160k, update notes"
+    (at 17.78 190.5 0)
+    (effects (font (size 1.27 1.27)) (justify left bottom))
+  )

Commit message: Rev 2.1
Updated to:
* Fit HP67 (reduced length/width, contact size/position)
* Board shape has 1mm recess on all four sides (better case design)
* All components fit on top side
* V2.1: slightly better thermal arrangement for regulator
Parts:
- BT1: footprint Connector_JST:JST_PH_B2B-PH-K_1x02_P2.00mm_Vertical -> Connector_PinHeader_2.00mm:PinHeader_1x02_P2.00mm_Vertical
- D1, D5: value 1N5819 -> 1N5817
- D2: value 5V1 -> 5V6; footprint Diode_SMD:D_SOD-123 -> Diode_SMD:D_SMA
- J2, J3: footprint george:PAD_10x12 -> george:PAD_10x15
- R1: value 4k -> 3k9
- R5: value 160k -> 150k
- R8: value 20k -> 24k
Other:
- note added: "BATTERY R1 ICHG TCHG R8 ICHG TCHG TRUN (USB) (USB) (HP) (HP) 2000 mAh 3k0 400mA 5H 24k 44mA 45H 1500 mAh 3k9 308mA 5H 24k 43mA 35H 16h (see spreadsheet) 1000 mAh 5k6 214mA 5H 22k 43mA 23H"
- note added: "REV1 - add Q1,R8,R9 REV2 - R1,R8 value"
- note added: "REV1 ADD Q1,R8,R9 REV1.1 U2=TPS73101, U4=S-8261ABJMD, R4=300k, R5=160k, update notes REV1.2 change D1 to 1N5817, change D2 to 5V6, R8=24k, Add C6 REV2 BOARD LAYOUT CHANGE"
- note added: "REV2 D1 to 1N5817"
- note removed: "BATTERY R1 ICHG TCHG R8 ICHG TCHG TRUN (USB) (USB) (HP) (HP) 2000 mAh 3k0 400mA 5H 22k 48mA 42H 1500 mAh 3k9 308mA 5H 22k 46.3mA 33H 16h (see spreadsheet) 1000 mAh 5k6 214mA 5H 20k 46.9mA 22H"
- note removed: "REV1 - add Q1,R8,R9"
- note removed: "REV1 ADD Q1,R8,R9 REV1.1 U2=TPS73101, U4=S-8261ABJMD, R4=300k, R5=160k, update notes"
